File: Onboarding-II/Onboarding-II.kicad_sch (KiCad schematic)
At the start: 0 parts

Commit message: New PCB Done
Parts:
- added C1, C2: .1uF, Capacitor_SMD:C_0603_1608Metric_Pad1.08x0.95mm_HandSolder, symbol Device:C
- added C3: 10nF, Capacitor_SMD:C_0603_1608Metric_Pad1.08x0.95mm_HandSolder, symbol Device:C
- added C4: 2.2uF, Capacitor_SMD:C_0603_1608Metric_Pad1.08x0.95mm_HandSolder, symbol Device:C
- added H1, H2: MountingHole, MountingHole:MountingHole_3.2mm_M3, symbol Mechanical:MountingHole
- added IC1: ICM-20602, footprints:IAM20680HP, symbol ICM-20602:ICM-20602
- added J1: Conn_01x05_Pin, Connector_PinHeader_2.54mm:PinHeader_1x05_P2.54mm_Horizontal, symbol Connector:Conn_01x05_Pin
Connections:
- new net: C1.1, IC1.14 (REGOUT)
- new net +5V: J1.3 (Pin_3)
- new net 3.3 VDC: C2.1, C3.1, C4.1, IC1.1 (VDDIO), IC1.16 (VDD), J1.2 (Pin_2)
- new net CS: IC1.5 (CS)
- new net GND: C1.2, C2.2, C3.2, C4.2, IC1.10 (RESV_3), IC1.11 (RESV_4), IC1.12 (RESV_5), IC1.13 (GND), IC1.15 (RESV_6), IC1.8 (FSYNC), IC1.9 (RESV_2), J1.1 (Pin_1)
- new net INT: IC1.6 (INT)
- new net SA0: IC1.4 (SA0/SDO)
- new net SCL: IC1.2 (SCL/SPC), J1.4 (Pin_4)
- new net SDA: IC1.3 (SDA/SDI), J1.5 (Pin_5)
- no-connect marks 0 -> 1
