File: Onboarding-II/Onboarding-II.kicad_sch (KiCad schematic)
At the start: 0 parts

Commit message: finished onboarding
Parts:
- added C1: 4.7uF, Package_TO_SOT_SMD:SOT-23-6, symbol Device:C
- added C2: 100nF, Package_TO_SOT_SMD:SOT-23-6, symbol Device:C
- added H1, H2: MountingHole, MountingHole:MountingHole_2.1mm, symbol Mechanical:MountingHole
- added J1: Conn_01x05_Pin, Sensor_Distance:ST_VL53L1x, symbol Connector:Conn_01x05_Pin
- added U1: VL53L1CXV0FY1, Sensor_Distance:ST_VL53L1x, symbol Sensor_Distance:VL53L1CXV0FY1
Connections:
- new net +2.8V: C1.1, C2.1, U1.1 (AVDDVCSEL), U1.11 (AVDD)
- new net +3.3V: J1.1 (Pin_1)
- new net +5V: J1.2 (Pin_2)
- new net GND: C1.2, C2.2, J1.5 (Pin_5), U1.12 (GND), U1.2 (AVSSVCSEL), U1.3 (GND), U1.4 (GND), U1.6 (GND)
- new net SCL: J1.4 (Pin_4), U1.10 (SCL)
- new net SDA: J1.3 (Pin_3), U1.9 (SDA)
Other:
- note added: "5-Pin Connector Sys"
- note added: "Mounting Holes"
- note added: "VL53L4CD Sensor"

Commit message: updated PCB
Parts:
- C1, C2: footprint Package_TO_SOT_SMD:SOT-23-6 -> Capacitor_SMD:C_0603_1608Metric_Pad1.08x0.95mm_HandSolder
- J1: footprint Sensor_Distance:ST_VL53L1x -> Connector_PinHeader_2.54mm:PinHeader_1x05_P2.54mm_Horizontal
Changed lines of the file:
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@@
 			)
 		)
-		(property "Footprint" "Package_TO_SOT_SMD:SOT-23-6"
+		(property "Footprint" "Capacitor_SMD:C_0603_1608Metric_Pad1.08x0.95mm_HandSolder"
 			(at 68.2752 64.77 0)
 			(hide yes)
@@
 			)
 		)
-		(property "Footprint" "Sensor_Distance:ST_VL53L1x"
+		(property "Footprint" "Connector_PinHeader_2.54mm:PinHeader_1x05_P2.54mm_Horizontal"
 			(at 113.03 62.23 0)
 			(hide yes)
@@
 			)
 		)
-		(property "Footprint" "Package_TO_SOT_SMD:SOT-23-6"
+		(property "Footprint" "Capacitor_SMD:C_0603_1608Metric_Pad1.08x0.95mm_HandSolder"
 			(at 74.6252 64.77 0)
 			(hide yes)
