File: Onboarding-II/Onboarding-II.kicad_sch (KiCad schematic)
At the start: 0 parts

Commit message: Added gerber, drill, and BOM deliverables for Onboarding II files to review.
Parts:
- added C1: 100nF, Capacitor_SMD:C_0805_2012Metric, symbol Device:C
- added C2: 4.7µF, Capacitor_SMD:C_0805_2012Metric, symbol Device:C
- added H1, H2: MountingHole, MountingHole:MountingHole_3.2mm_M3, symbol Mechanical:MountingHole
- added IC1: VL53L4CDV0DH_1, footprints:VL53L4CDV0DH1, symbol VL53L4CDV0DH_1:VL53L4CDV0DH_1
- added J1: Conn_01x05_Pin, Connector_PinSocket_2.54mm:PinSocket_1x05_P2.54mm_Vertical, symbol Connector:Conn_01x05_Pin
- added R1, R2: 10kΩ, Resistor_SMD:R_0805_2012Metric, symbol Device:R
Connections:
- new net +3.3V: C1.1, C2.1, IC1.1 (AVDDVCSEL_1), IC1.11 (AVDD), IC1.13 (AVDDVCSEL_2), J1.1 (Pin_1), R1.1, R2.1
- new net 5V: J1.3 (Pin_3)
- new net GND: C1.2, C2.2, IC1.12 (GND4), IC1.2 (AVSSVCSEL), IC1.3 (GND), IC1.4 (GND2), IC1.6 (GND3), J1.5 (Pin_5)
- new net GPIO1: IC1.7 (GPIO1)
- new net SCL: IC1.10 (SCL), J1.4 (Pin_4), R2.2
- new net SDA: IC1.9 (SDA), J1.2 (Pin_2), R1.2
- new net XSHUT: IC1.5 (XSHUT)
- no-connect marks 0 -> 1
